File: driver.sch (KiCad schematic (older format))
At the start: 28 parts, among them J1 Conn_01x04, J2 Conn_01x02, J3 Conn_01x04, J4 Conn_01x04, J5 Conn_01x02, J6 Conn_01x02, J7 Conn_01x03, J8 Conn_01x04, U1 L6470H

Commit message: Update schematic
Parts:
- removed J7: Conn_01x03, Connector_PinHeader_2.54mm:PinHeader_1x03_P2.54mm_Horizontal, symbol Connector_Generic:Conn_01x03
- added JP1: SolderJumper_3_Open, Jumper:SolderJumper-3_P1.3mm_Open_RoundedPad1.0x1.5mm_NumberLabels, symbol Jumper:SolderJumper_3_Open
Connections:
- net +5V: now also JP1.3 (B)
- net VDD: now also JP1.2 (C)
- net at U1.6 (VREG): now also JP1.1 (A)
Changed lines of the file:
@@
 	6100 2200 6100 2300
 Wire Wire Line
-	5400 2300 5400 2100
-$Comp
-L Connector_Generic:Conn_01x03 J7
-U 1 1 5D9A30B9
-P 4900 2100
-F 0 "J7" H 4818 1867 50  0000 C CNN
-F 1 "Conn_01x03" H 4818 1866 50  0001 C CNN
-F 2 "Connector_PinHeader_2.54mm:PinHeader_1x03_P2.54mm_Horizontal" H 4900 2100 50  0001 C CNN
-F 3 "~" H 4900 2100 50  0001 C CNN
-	1    4900 2100
-	-1   0    0    1
-$EndComp
-Wire Wire Line
-	5100 2200 5300 2200
-Wire Wire Line
-	5300 2200 5300 2300
+	5400 2300 5400 2000
 $Comp
 L power:+5V #PWR010
 U 1 1 5D9A427F
-P 5200 1950
-F 0 "#PWR010" H 5200 1800 50  0001 C CNN
-F 1 "+5V" H 5215 2123 50  0000 C CNN
-F 2 "" H 5200 1950 50  0001 C CNN
-F 3 "" H 5200 1950 50  0001 C CNN
-	1    5200 1950
-	1    0    0    -1
-$EndComp
-Wire Wire Line
-	5200 1950 5200 2000
-Wire Wire Line
-	5200 2000 5100 2000
+P 4950 1700
+F 0 "#PWR010" H 4950 1550 50  0001 C CNN
+F 1 "+5V" H 4965 1873 50  0000 C CNN
+F 2 "" H 4950 1700 50  0001 C CNN
+F 3 "" H 4950 1700 50  0001 C CNN
+	1    4950 1700
+	1    0    0    -1
+$EndComp
 $Comp
 L Device:R R1
@@
 L power:VDD #PWR011
 U 1 1 5D9A704D
-P 5400 1950
-F 0 "#PWR011" H 5400 1800 50  0001 C CNN
-F 1 "VDD" H 5417 2123 50  0000 C CNN
-F 2 "" H 5400 1950 50  0001 C CNN
-F 3 "" H 5400 1950 50  0001 C CNN
-	1    5400 1950
-	1    0    0    -1
-$EndComp
-Wire Wire Line
-	5400 1950 5400 2100
-Connection ~ 5400 2100
+P 5400 1900
+F 0 "#PWR011" H 5400 1750 50  0001 C CNN
+F 1 "VDD" H 5417 2073 50  0000 C CNN
+F 2 "" H 5400 1900 50  0001 C CNN
+F 3 "" H 5400 1900 50  0001 C CNN
+	1    5400 1900
+	1    0    0    -1
+$EndComp
+Wire Wire Line
+	5400 1900 5400 2000
+Connection ~ 5400 2000
 $Comp
 L power:VDD #PWR09
@@
 Connection ~ 6100 2200
 Wire Wire Line
-	5100 2100 5400 2100
+	5100 2000 5400 2000
 $Comp
 L Driver_stepper_ST:L6470H U1
@@
 Wire Wire Line
 	4100 2650 4100 2750
+$Comp
+L Jumper:SolderJumper_3_Open JP1
+U 1 1 5DBF9C5D
+P 4950 2000
+F 0 "JP1" V 4950 2068 50  0000 L CNN
+F 1 "SolderJumper_3_Open" V 4905 2067 50  0001 L CNN
+F 2 "Jumper:SolderJumper-3_P1.3mm_Open_RoundedPad1.0x1.5mm_NumberLabels" H 4950 2000 50  0001 C CNN
+F 3 "~" H 4950 2000 50  0001 C CNN
+	1    4950 2000
+	0    -1   -1   0
+$EndComp
+Wire Wire Line
+	4950 1700 4950 1800
+Wire Wire Line
+	4950 2200 4950 2250
+Wire Wire Line
+	4950 2250 5300 2250
+Wire Wire Line
+	5300 2250 5300 2300
 $EndSCHEMATC
