File: driver.sch (KiCad schematic (older format))
At the start: 30 parts, among them J1 Conn_01x04, J2 Conn_01x02, J3 Conn_01x04, J4 Conn_01x04, J5 Conn_01x02, J6 Conn_01x02, J7 Conn_01x04, U1 L6470H

Commit message: Assign values
Parts:
- C1: value CP -> 100.0; Voltage (none) -> 63V
- C2, C4: value C -> 0.22; Voltage (none) -> 50V
- C3: value CP -> 10.0; Voltage (none) -> 16V
- C5: value C -> 0.1
- C6: value C -> 0.22
- C7: value C -> 0.01
- D2, D3, D4: value LED -> FYLS - 0805UGC
- R1, R3: value R -> 10k
- R2: value R -> 10k; Note (none) -> Attenuation is needed
- R4: value R -> 62k
- R5: value R -> 2k7
- R6, R7, R8: value R -> 240
Other:
- moved on the sheet: C2, C4
Changed lines of the file:
@@
 P 5800 1700
 F 0 "C7" H 5915 1746 50  0000 L CNN
-F 1 "C" H 5915 1655 50  0000 L CNN
+F 1 "0.01" H 5915 1655 50  0000 L CNN
 F 2 "Capacitor_SMD:C_0805_2012Metric" H 5838 1550 50  0001 C CNN
 F 3 "~" H 5800 1700 50  0001 C CNN
@@
 P 5800 1100
 F 0 "C6" V 5548 1100 50  0000 C CNN
-F 1 "C" V 5639 1100 50  0000 C CNN
+F 1 "0.22" V 5639 1100 50  0000 C CNN
 F 2 "Capacitor_SMD:C_0805_2012Metric" H 5838 950 50  0001 C CNN
 F 3 "~" H 5800 1100 50  0001 C CNN
@@
 P 4100 2500
 F 0 "R1" H 4170 2546 50  0000 L CNN
-F 1 "R" H 4170 2455 50  0000 L CNN
+F 1 "10k" H 4170 2455 50  0000 L CNN
 F 2 "Resistor_SMD:R_0805_2012Metric" V 4030 2500 50  0001 C CNN
 F 3 "~" H 4100 2500 50  0001 C CNN
@@
 P 4500 2500
 F 0 "R3" H 4570 2546 50  0000 L CNN
-F 1 "R" H 4570 2455 50  0000 L CNN
+F 1 "10k" H 4570 2455 50  0000 L CNN
 F 2 "Resistor_SMD:R_0805_2012Metric" V 4430 2500 50  0001 C CNN
 F 3 "~" H 4500 2500 50  0001 C CNN
@@
 P 1700 1350
 F 0 "C1" H 1818 1396 50  0000 L CNN
-F 1 "CP" H 1818 1305 50  0000 L CNN
+F 1 "100.0" H 1818 1305 50  0000 L CNN
 F 2 "Capacitor_THT:CP_Radial_D10.0mm_P5.00mm" H 1738 1200 50  0001 C CNN
 F 3 "~" H 1700 1350 50  0001 C CNN
+F 4 "63V" H 1900 1200 50  0000 C CNN "Voltage"
 	1    1700 1350
 	1    0    0    -1
@@
 P 7250 2500
 F 0 "R4" H 7320 2546 50  0000 L CNN
-F 1 "R" H 7320 2455 50  0000 L CNN
+F 1 "62k" H 7320 2455 50  0000 L CNN
 F 2 "Resistor_SMD:R_0805_2012Metric" V 7180 2500 50  0001 C CNN
 F 3 "~" H 7250 2500 50  0001 C CNN
@@
 P 7250 3000
 F 0 "R5" H 7320 3046 50  0000 L CNN
-F 1 "R" H 7320 2955 50  0000 L CNN
+F 1 "2k7" H 7320 2955 50  0000 L CNN
 F 2 "Resistor_SMD:R_0805_2012Metric" V 7180 3000 50  0001 C CNN
 F 3 "~" H 7250 3000 50  0001 C CNN
@@
 L Device:C C4
 U 1 1 5D9B36C7
-P 3150 1350
-F 0 "C4" H 3265 1396 50  0000 L CNN
-F 1 "C" H 3265 1305 50  0000 L CNN
-F 2 "Capacitor_SMD:C_0805_2012Metric" H 3188 1200 50  0001 C CNN
-F 3 "~" H 3150 1350 50  0001 C CNN
-	1    3150 1350
+P 3400 1350
+F 0 "C4" H 3515 1396 50  0000 L CNN
+F 1 "0.22" H 3515 1305 50  0000 L CNN
+F 2 "Capacitor_SMD:C_0805_2012Metric" H 3438 1200 50  0001 C CNN
+F 3 "~" H 3400 1350 50  0001 C CNN
+F 4 "50V" H 3600 1200 50  0000 C CNN "Voltage"
+	1    3400 1350
 	1    0    0    -1
 $EndComp
@@
 P 2800 1350
 F 0 "C3" H 2918 1396 50  0000 L CNN
-F 1 "CP" H 2918 1305 50  0000 L CNN
+F 1 "10.0" H 2918 1305 50  0000 L CNN
 F 2 "Capacitor_Tantalum_SMD:CP_EIA-3216-18_Kemet-A" H 2838 1200 50  0001 C CNN
 F 3 "~" H 2800 1350 50  0001 C CNN
+F 4 "16V" H 3000 1200 50  0000 C CNN "Voltage"
 	1    2800 1350
 	1    0    0    -1
@@
 L power:VDD #PWR05
 U 1 1 5D9B3D5A
-P 3150 1000
-F 0 "#PWR05" H 3150 850 50  0001 C CNN
-F 1 "VDD" H 3167 1173 50  0000 C CNN
-F 2 "" H 3150 1000 50  0001 C CNN
-F 3 "" H 3150 1000 50  0001 C CNN
-	1    3150 1000
+P 3400 1000
+F 0 "#PWR05" H 3400 850 50  0001 C CNN
+F 1 "VDD" H 3417 1173 50  0000 C CNN
+F 2 "" H 3400 1000 50  0001 C CNN
+F 3 "" H 3400 1000 50  0001 C CNN
+	1    3400 1000
 	1    0    0    -1
 $EndComp
@@
 	2800 1200 2800 1100
 Wire Wire Line
-	3150 1000 3150 1100
-Wire Wire Line
-	2800 1100 3150 1100
-Connection ~ 3150 1100
-Wire Wire Line
-	3150 1100 3150 1200
+	3400 1000 3400 1100
+Wire Wire Line
+	2800 1100 3400 1100
+Connection ~ 3400 1100
+Wire Wire Line
+	3400 1100 3400 1200
 Wire Wire Line
 	2800 1500 2800 1600
 Wire Wire Line
-	2800 1600 3150 1600
-Wire Wire Line
-	3150 1600 3150 1500
+	2800 1600 3400 1600
+Wire Wire Line
+	3400 1600 3400 1500
 $Comp
 L power:GNDD #PWR06
 U 1 1 5D9B81CE
-P 3150 1700
-F 0 "#PWR06" H 3150 1450 50  0001 C CNN
-F 1 "GNDD" H 3154 1545 50  0000 C CNN
-F 2 "" H 3150 1700 50  0001 C CNN
-F 3 "" H 3150 1700 50  0001 C CNN
-	1    3150 1700
-	1    0    0    -1
-$EndComp
-Wire Wire Line
-	3150 1700 3150 1600
-Connection ~ 3150 1600
+P 3400 1700
+F 0 "#PWR06" H 3400 1450 50  0001 C CNN
+F 1 "GNDD" H 3404 1545 50  0000 C CNN
+F 2 "" H 3400 1700 50  0001 C CNN
+F 3 "" H 3400 1700 50  0001 C CNN
+	1    3400 1700
+	1    0    0    -1
+$EndComp
+Wire Wire Line
+	3400 1700 3400 1600
+Connection ~ 3400 1600
 $Comp
 L power:GND #PWR013
@@
 L power:VCC #PWR03
 U 1 1 5D9FA699
-P 2100 1000
-F 0 "#PWR03" H 2100 850 50  0001 C CNN
-F 1 "VCC" H 2117 1173 50  0000 C CNN
-F 2 "" H 2100 1000 50  0001 C CNN
-F 3 "" H 2100 1000 50  0001 C CNN
-	1    2100 1000
+P 2200 1000
+F 0 "#PWR03" H 2200 850 50  0001 C CNN
+F 1 "VCC" H 2217 1173 50  0000 C CNN
+F 2 "" H 2200 1000 50  0001 C CNN
+F 3 "" H 2200 1000 50  0001 C CNN
+	1    2200 1000
 	-1   0    0    -1
 $EndComp
@@
 L power:GND #PWR04
 U 1 1 5D9FAE42
-P 2100 1700
-F 0 "#PWR04" H 2100 1450 50  0001 C CNN
-F 1 "GND" H 2105 1527 50  0000 C CNN
-F 2 "" H 2100 1700 50  0001 C CNN
-F 3 "" H 2100 1700 50  0001 C CNN
-	1    2100 1700
+P 2200 1700
+F 0 "#PWR04" H 2200 1450 50  0001 C CNN
+F 1 "GND" H 2205 1527 50  0000 C CNN
+F 2 "" H 2200 1700 50  0001 C CNN
+F 3 "" H 2200 1700 50  0001 C CNN
+	1    2200 1700
 	-1   0    0    -1
 $EndComp
@@
 P 10350 1850
 F 0 "D4" V 10343 1732 50  0000 R CNN
-F 1 "LED" V 10298 1733 50  0001 R CNN
+F 1 "FYLS - 0805UGC" V 10298 1733 50  0001 R CNN
 F 2 "LED_SMD:LED_0805_2012Metric" H 10350 1850 50  0001 C CNN
 F 3 "~" H 10350 1850 50  0001 C CNN
@@
 P 10350 1450
 F 0 "R8" H 10420 1496 50  0000 L CNN
-F 1 "R" H 10420 1405 50  0000 L CNN
+F 1 "240" H 10420 1405 50  0000 L CNN
 F 2 "Resistor_SMD:R_0805_2012Metric" V 10280 1450 50  0001 C CNN
 F 3 "~" H 10350 1450 50  0001 C CNN
@@
 P 9650 1850
 F 0 "D2" V 9643 1732 50  0000 R CNN
-F 1 "LED" V 9598 1733 50  0001 R CNN
+F 1 "FYLS - 0805UGC" V 9598 1733 50  0001 R CNN
 F 2 "LED_SMD:LED_0805_2012Metric" H 9650 1850 50  0001 C CNN
 F 3 "~" H 9650 1850 50  0001 C CNN
@@
 P 9650 1450
 F 0 "R6" H 9720 1496 50  0000 L CNN
-F 1 "R" H 9720 1405 50  0000 L CNN
+F 1 "240" H 9720 1405 50  0000 L CNN
 F 2 "Resistor_SMD:R_0805_2012Metric" V 9580 1450 50  0001 C CNN
 F 3 "~" H 9650 1450 50  0001 C CNN
@@
 P 10000 1850
 F 0 "D3" V 9993 1732 50  0000 R CNN
-F 1 "LED" V 9948 1733 50  0001 R CNN
+F 1 "FYLS - 0805UGC" V 9948 1733 50  0001 R CNN
 F 2 "LED_SMD:LED_0805_2012Metric" H 10000 1850 50  0001 C CNN
 F 3 "~" H 10000 1850 50  0001 C CNN
@@
 P 10000 1450
 F 0 "R7" H 10070 1496 50  0000 L CNN
-F 1 "R" H 10070 1405 50  0000 L CNN
+F 1 "240" H 10070 1405 50  0000 L CNN
 F 2 "Resistor_SMD:R_0805_2012Metric" V 9930 1450 50  0001 C CNN
 F 3 "~" H 10000 1450 50  0001 C CNN
@@
 L Device:C C2
 U 1 1 5D9AA958
-P 2100 1350
-F 0 "C2" H 2215 1396 50  0000 L CNN
-F 1 "C" H 2215 1305 50  0000 L CNN
-F 2 "Capacitor_SMD:C_0805_2012Metric" H 2138 1200 50  0001 C CNN
-F 3 "~" H 2100 1350 50  0001 C CNN
-	1    2100 1350
-	1    0    0    -1
-$EndComp
-Wire Wire Line
-	2100 1200 2100 1100
-Wire Wire Line
-	2100 1100 1700 1100
+P 2200 1350
+F 0 "C2" H 2315 1396 50  0000 L CNN
+F 1 "0.22" H 2315 1305 50  0000 L CNN
+F 2 "Capacitor_SMD:C_0805_2012Metric" H 2238 1200 50  0001 C CNN
+F 3 "~" H 2200 1350 50  0001 C CNN
+F 4 "50V" H 2400 1200 50  0000 C CNN "Voltage"
+	1    2200 1350
+	1    0    0    -1
+$EndComp
+Wire Wire Line
+	2200 1200 2200 1100
+Wire Wire Line
+	2200 1100 1700 1100
 Wire Wire Line
 	1700 1200 1700 1100
@@
 	1500 1600 1700 1600
 Wire Wire Line
-	2100 1600 2100 1500
+	2200 1600 2200 1500
 Wire Wire Line
 	1700 1500 1700 1600
 Connection ~ 1700 1600
 Wire Wire Line
-	1700 1600 2100 1600
-Wire Wire Line
-	2100 1000 2100 1100
-Connection ~ 2100 1100
-Wire Wire Line
-	2100 1700 2100 1600
-Connection ~ 2100 1600
+	1700 1600 2200 1600
+Wire Wire Line
+	2200 1000 2200 1100
+Connection ~ 2200 1100
+Wire Wire Line
+	2200 1700 2200 1600
+Connection ~ 2200 1600
 Wire Wire Line
 	5800 2300 5800 1850
@@
 P 4450 3750
 F 0 "R2" V 4550 3800 50  0000 L CNN
-F 1 "R" V 4550 3600 50  0000 L CNN
+F 1 "10k" V 4550 3600 50  0000 L CNN
 F 2 "Resistor_SMD:R_0805_2012Metric" V 4380 3750 50  0001 C CNN
 F 3 "~" H 4450 3750 50  0001 C CNN
+F 4 "Attenuation is needed" V 4450 3750 50  0001 C CNN "Note"
 	1    4450 3750
 	0    -1   -1   0
@@
 P 4150 4000
 F 0 "C5" H 4265 4046 50  0000 L CNN
-F 1 "C" H 4265 3955 50  0000 L CNN
+F 1 "0.1" H 4265 3955 50  0000 L CNN
 F 2 "Capacitor_SMD:C_0805_2012Metric" H 4188 3850 50  0001 C CNN
 F 3 "~" H 4150 4000 50  0001 C CNN

Commit message: REV 1.0
Parts:
- D1: symbol Diode:BAV99 -> driver-rescue:BAV99-Diode
Changed lines of the file:
@@
 EESchema Schematic File Version 4
-LIBS:driver-cache
 EELAYER 30 0
 EELAYER END
@@
 $EndDescr
 $Comp
-L Diode:BAV99 D1
+L driver-rescue:BAV99-Diode D1
 U 2 1 5D9A9BF0
 P 5550 1450
@@
 $EndComp
 $Comp
-L Diode:BAV99 D1
+L driver-rescue:BAV99-Diode D1
 U 1 1 5D9A9FF3
 P 6050 1450
