File: driver.kicad_pcb (KiCad board)
At the start: 2 copper layers, 50 x 50 mm, 28 parts, among them J1 Conn_01x04, J2 Conn_01x02, J3 Conn_01x04, J4 Conn_01x04, J5 Conn_01x02, J6 Conn_01x02, J7 Conn_01x03, J8 Conn_01x04, U1 L6470H

Commit message: PCB
Parts:
- removed J7: Conn_01x03, Connector_PinHeader_2.54mm:PinHeader_1x03_P2.54mm_Horizontal
- added JP1: SolderJumper_3_Open, Jumper:SolderJumper-3_P1.3mm_Open_RoundedPad1.0x1.5mm_NumberLabels, F.Cu at (99.5, 59.8)
- C5, R1, R3, R4, R5, R6, R7: moved to B.Cu
- moved R8 37.1 mm to (78.1, 62.0), turned to 180 degrees
- moved D4 36.5 mm to (78.1, 59.0), turned to 180 degrees
- moved J6 28.0 mm to (101.0, 54.5), turned to 0 degrees
- moved D2 9.03 mm to (98.0, 31.0), turned to 90 degrees
- moved R6 8.57 mm to (98.0, 30.9), turned to 90 degrees
- moved R1 8.50 mm to (97.4, 36.5)
- moved R5 6.02 mm to (88.5, 52.5)
- moved C3 5.83 mm to (94.8, 41.0), turned to 180 degrees
- moved R3 5.51 mm to (97.4, 38.5)
- moved C4 5.41 mm to (94.0, 38.5), turned to 180 degrees
- moved D3 3.05 mm to (101.0, 31.0), turned to 90 degrees
- moved C7 2.95 mm to (90.0, 51.0)
- moved R4 2.86 mm to (86.5, 52.5)
- moved C6 2.85 mm to (93.1, 49.0)
- moved D1 2.70 mm to (93.0, 52.0)
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Routing:
- net VDD: track 0.00 -> 73.7 mm, vias 0 -> 2
- net GND: track 28.7 -> 94.3 mm
- net /~BUSY: track 0.00 -> 43.6 mm, vias 0 -> 1
- net Net-(J3-Pad4): track 0.00 -> 32.7 mm, vias 0 -> 1
- net /~FLAG: track 0.00 -> 32.6 mm, vias 0 -> 1
- net VCC: track 41.1 -> 73.5 mm, vias 4 -> 8
- net Net-(J3-Pad3): track 0.00 -> 32.4 mm, vias 0 -> 1
- net Net-(R2-Pad2): track 0.00 -> 25.6 mm, vias 0 -> 2
- net Net-(J4-Pad3): track 0.00 -> 24.0 mm, vias 0 -> 1
- net Net-(J4-Pad4): track 0.00 -> 22.8 mm, vias 0 -> 1
- net Net-(JP1-Pad1): track 0.00 -> 22.6 mm
- net Net-(J4-Pad2): track 0.00 -> 22.5 mm, vias 0 -> 1
- net Net-(J6-Pad2): track 0.00 -> 20.9 mm
- net Net-(J6-Pad1): track 0.00 -> 20.8 mm
- net Net-(J4-Pad1): track 0.00 -> 20.1 mm, vias 0 -> 1
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- added copper zone on F.Cu, net VCC
- removed copper zone on F.Cu, net Net-(J8-Pad1)
- removed copper zone on F.Cu, net Net-(J8-Pad2)
- removed copper zone on F.Cu, net Net-(J8-Pad3)
- removed copper zone on F.Cu, net Net-(J8-Pad4)

Commit message: Silkscreen
Parts:
- added H1: MountingHole, MountingHole:MountingHole_3.2mm_M3, F.Cu at (73.0, 65.0)
- added H2: MountingHole, MountingHole:MountingHole_3.2mm_M3, F.Cu at (101.0, 25.5)
- moved D2 0.50 mm to (98.0, 31.5)
- moved D3 0.50 mm to (101.0, 31.5)
- moved R6 0.50 mm to (98.0, 31.4)
- moved R7 0.50 mm to (101.0, 31.4)
- renumbered J8 to J7
Routing:
- net VDD: track 73.7 -> 73.2 mm
- net /~FLAG: track 32.6 -> 32.1 mm
- net /~BUSY: track 43.6 -> 43.1 mm
Other:
- board size 50 x 50 mm -> 36.5 x 48 mm
- board text added: "+5"
- board text added: "A1"
- board text added: "A2"
- board text added: "B1"
- board text added: "B2"
- board text added: "GND"
- board text added: "Vcc"
- board text added: "Vdd"
- board text added: "ext"
- board text added: "flag"
- board text added: "int"
- board text added: "l6470 driver REV 1.0"
- board text added: "sync"

Commit message: REV 1.0
Parts:
- moved R7 6.17 mm to (95.0, 30.0), turned to 0 degrees
- moved R6 3.05 mm to (95.0, 32.0), turned to 0 degrees
- moved D2 3.00 mm to (98.0, 34.5)
- moved D3 3.00 mm to (101.0, 34.5)
- moved H2 2.50 mm to (101.0, 28.0)
- moved D4 2.12 mm to (79.6, 57.5)
- moved R2 2.05 mm to (75.0, 34.5)
- moved H1 2.00 mm to (75.0, 65.0)
- moved J4 2.00 mm to (75.0, 39.5)
- moved J5 2.00 mm to (75.0, 30.6)
- moved R8 1.58 mm to (79.6, 61.5)
- moved C5 1.56 mm to (76.1, 33.0)
Routing:
- net /~BUSY: track 43.1 -> 31.7 mm
- net VDD: track 73.2 -> 65.4 mm
- net GND: track 94.3 -> 98.8 mm
- net Net-(D3-Pad2): track 3.06 -> 7.45 mm
- net /~FLAG: track 32.1 -> 28.9 mm
- net Net-(J4-Pad2): track 22.5 -> 20.4 mm
- net Net-(J4-Pad3): track 24.0 -> 22.0 mm
- net Net-(J4-Pad4): track 22.8 -> 21.2 mm
- net Net-(R2-Pad2): track 25.6 -> 24.1 mm
- net Net-(J4-Pad1): track 20.1 -> 19.0 mm
- net Net-(D4-Pad2): track 3.00 -> 4.00 mm
- net Net-(J3-Pad4): track 32.7 -> 31.8 mm
- net Net-(JP1-Pad1): track 22.6 -> 23.4 mm
- net Net-(D2-Pad2): track 3.06 -> 3.59 mm
Other:
- board size 36.5 x 48 mm -> 35 x 45 mm
- board text added: "L6470 driver REV 1.0"
- board text removed: "l6470 driver REV 1.0"
